File: Light_intensity_data_logger/Light_intensity_data_logger.kicad_pcb (KiCad board)
At the start: 2 copper layers, 105 x 69 mm, 24 parts, among them J1 Wire_to_Vbat, Q1 NTJD4001NT1G, Q2 NTJD4001NT1G, U1 BME280, U2 TCS34725FN, U3 TSL25911FN, U4 Teensy3.6

Commit message: License info and annotations added
Parts:
- added REF**: CC_Attribution, Ben_Custom:CC_Attribution, F.Cu at (156.1, 98.6)
- added REF**: CC_Share_alike, Ben_Custom:CC_Share_alike, F.Cu at (151.3, 98.6)
- added REF**: CC silkscreen, Ben_Custom:CC_silkscreen, F.Cu at (146.3, 98.5)
- moved REF*** 2.67 mm to (151.2, 90.4)
- moved R1 0.72 mm to (150.5, 63.6)
- moved BT1 0.18 mm to (114.0, 51.8)
- renumbered C3 to C2, C2 to C3
Connections:
- net /21* renamed Net-(U4-Pad48)
- net /22* renamed Net-(U4-Pad49)
- net /34 renamed Net-(U4-Pad31)
- net /35 renamed Net-(U4-Pad32)
Routing:
- net GND: track 429.6 -> 434.1 mm
- net Net-(LCD1-Pad15): track 6.21 -> 7.03 mm
- net Net-(Q1-Pad4): track 77.8 -> 77.2 mm
Other:
- board text added: "1 8"
- board text added: "3.6V min 6.0V max"
- board text added: "9 16"
- board text added: "Designed by Benjamin E. Smith Funded by NIH P30-EY003176-32 https://github.com/Llamero/Light_Color_and_Intensity_Datalogger"
- board text added: "Wire to Vbat"

Commit message: Removed extra ground trace
Routing:
- net GND: track 434.1 -> 428.5 mm
Changed lines of the file:
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@@
     (thickness 1.6)
     (drawings 46)
-    (tracks 1385)
+    (tracks 1386)
     (zones 0)
     (modules 27)
@@
   (segment (start 113.230001 84.8448) (end 113.23 84.301899) (width 0.2) (layer F.Cu) (net 2))
   (segment (start 113.23 84.301899) (end 113.23 84.16) (width 0.2) (layer F.Cu) (net 2))
-  (segment (start 111.49 84.16) (end 106.71 88.94) (width 0.25) (layer F.Cu) (net 2))
   (segment (start 106.71 88.94) (end 106.67 88.94) (width 0.25) (layer F.Cu) (net 2))
   (segment (start 111.49 84.16) (end 113.23 84.16) (width 0.25) (layer F.Cu) (net 2))
@@
   (segment (start 149.71 64.89) (end 144.85 69.75) (width 0.25) (layer F.Cu) (net 2))
   (segment (start 144.81 69.75) (end 143.41 71.15) (width 0.25) (layer F.Cu) (net 2))
+  (segment (start 111.49 84.16) (end 111.26999 84.38001) (width 0.25) (layer F.Cu) (net 2))
+  (segment (start 111.26999 84.38001) (end 110.64 85.01) (width 0.25) (layer F.Cu) (net 2))
   (segment (start 99 45.05) (end 93.23 45.05) (width 1) (layer F.Cu) (net 3))
   (segment (start 93.23 45.05) (end 93.31 45.13) (width 1) (layer F.Cu) (net 3))
